File: circuit/Main circuit V1.0/Main circuit V1.0.kicad_sch (KiCad schematic)
At the start: 35 parts, among them J1 Power IN, J10 AdapterOut, J11 AdapterIN, J2 Fan Out, J4 UnihikerK10_connector, J5 Light Out 2, J6 LeftTopTouch, J7 LeftBottomTouch, J8 RightTopTouch, J9 RightBottomTouch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

Commit message: fan speed, alarm timeout added
Parts:
- added R2: 2.2k, Resistor_SMD:R_1206_3216Metric, symbol Device:R
Connections:
- new net LCD_BLK: R2.2
- new net P1: R2.1
Other:
- note added: "Comments: All touch sensors have 15pF capacitors additionally connected from touch pad to gnd, to adjust for sensitivity."
- note added: "Comments: Do not use 104j since low power leds might glow dimly when not signalled"
- note added: "Comments: P0 and P1 are direct pins of ESP32, used here for LEDC capability used for backlight control and IR led control"
- note removed: "Do not use 104j since low power leds might glow dimly when not signalled"
- company: (none) -> Al Amin Ashik
- title: ATH B1 -> Home automation socket
- moved on the sheet: C1, C2, C4, C7, C8, D5, J1, J10, J11, J2, J4, J5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
